File: NAVCORE-SoOP.kicad_pcb (KiCad board)
At the start: 6 copper layers, 45 x 47.2 mm, 190 parts, among them J1 USB-C, J11 SERIAL2 4P, J12 U.FL ANT, J14 FLOW 6P, J15 LED 3P, J16 BUZZ 2P, J17 SERVO 6P, J18 PYRO 2P, J19 SWD 4P, J2 ESC 8P, J20 TOUCH 2P, J3 GPS+I2C, J5 RC IN, J6 CAN 4P, J8 microSD, J9 I2C 4P, P41 TEL_5V, P44 TEL_PPS, P46 TEL_GND, P71 RF_5V, P72 RF_TX, P73 RF_RX, P74 RF_GND, Q1 AO3400A, Q3 AO3400A, Q4 WST4041, Q5 AO3400A, SW1 BOOT, SW2 RESET, U1 STM32H743VIT6, U10 TLV75533, U11 SN65HVD230, U12 USBLC6-2SC6, U13 MAX2112, U14 OPA2374, U17 74LVC1G17, U19 TMP119, U2 ICM-42688-P, U20 LMR33630A, U21 XC6206P332MR, U3 ICM-42605, U4 MS5611, U5 W25Q128JVSIQ, U8 LMR33630A, U9 AP2112K-3.3, Y1 8MHz, Y2 25MHz TCXO

Commit message: Fix the tuner loop filter and IMU chip select, mark the forward edge
Parts:
- added C81: 1n, Capacitor_SMD:C_0402_1005Metric, F.Cu at (142.2, 122.7)
- added C84: 1n, Capacitor_SMD:C_0402_1005Metric, F.Cu at (141.5, 113.9)
- added C86: 1n, Capacitor_SMD:C_0402_1005Metric, F.Cu at (143.0, 116.4)
- added R57: 470R, Resistor_SMD:R_0402_1005Metric, F.Cu at (142.8, 121.4)
- added R58: 4k7, Resistor_SMD:R_0402_1005Metric, B.Cu at (143.0, 109.2)
- C56: value 10n -> 100p
- C57: value 10n -> 100n
- R34: value 1k -> 330R
Routing:
- net VCC_RF: track 27.5 -> 36.0 mm, vias 0 -> 2
- net CPOUT: track 1.66 -> 6.42 mm, vias 0 -> 1
- net VTUNE: track 2.06 -> 6.44 mm, vias 0 -> 1
- net GC1: track 3.84 -> 7.00 mm, vias 0 -> 2

Commit message: give the payload and analogue rails real copper, put C41 on the CAN supply
Connections:
- C41 pad 1: +3V3 -> +3V3_CAN
Routing:
- net +3V3: track 174.7 -> 169.5 mm
- net +5V: track 125.7 -> 121.6 mm
- net +5V_PAYLOAD: track 129.9 -> 127.0 mm
- net +3V3A: track 122.0 -> 120.4 mm
- net +3V3_CAN: track 10.8 -> 12.2 mm
- net VBAT: track 79.2 -> 78.4 mm
Changed lines of the file:
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@@
 		(property "Reference" "C75"
 			(at -1.51 -0.31 90)
-			(layer "F.SilkS")
+			(layer "F.Fab")
 			(effects
 				(font
@@
 		(property "Reference" "R51"
 			(at 0 -1.17 0)
-			(layer "F.SilkS")
+			(layer "F.Fab")
 			(effects
 				(font
@@
 			(layers "B.Cu" "B.Mask" "B.Paste")
 			(roundrect_rratio 0.25)
-			(net 5 "+3V3")
+			(net 140 "+3V3_CAN")
 		)
 		(pad "2" smd roundrect
@@
 		(property "Reference" "C74"
 			(at 0 1.16 0)
-			(layer "B.SilkS")
+			(layer "B.Fab")
 			(effects
 				(font
@@
 		(property "Reference" "C76"
 			(at 0 1.16 0)
-			(layer "B.SilkS")
+			(layer "B.Fab")
 			(effects
 				(font
@@
 		(property "Reference" "F1"
 			(at 0 1.83 270)
-			(layer "B.SilkS")
+			(layer "B.Fab")
 			(effects
 				(font
@@
 	(segment
 		(start 129.28125 117.11875)
-		(end 129.28125 115.93125)
+		(end 129.5398 116.439858)
 		(width 0.1016)
 		(layer "B.Cu")
@@
 	)
 	(segment
-		(start 129.28125 115.93125)
-		(end 129.53125 115.93125)
-		(width 0.1016)
-		(layer "B.Cu")
-		(net 3)
-	)
-	(segment
 		(start 104.1041 105)
 		(end 104.1863 105.0822)
@@
 	)
 	(segment
-		(start 104.53125 124.93125)
-		(end 104.59375 124.93125)
-		(width 0.1016)
-		(layer "In3.Cu")
-		(net 3)
-	)
-	(segment
 		(start 104.90625 113.24375)
 		(end 104.96875 113.24375)
@@
 	)
 	(segment
-		(start 124.4915 143.7511)
+		(start 123.800102 143.751062)
 		(end 123.096 143.7511)
 		(width 0.1016)
@@
 	)
 	(segment
-		(start 126.6801 143.7511)
-		(end 127.432963 144.185765)
-		(width 0.25)
-		(layer "F.Cu")
-		(net 4)
-	)
-	(segment
 		(start 140.2991 125.4171)
 		(end 140.1566 125.5596)
@@
 	)
 	(segment
-		(start 131.605006 128.919998)
-		(end 131.605006 130.272987)
-		(width 0.25)
-		(layer "F.Cu")
-		(net 4)
-	)
-	(segment
 		(start 130.8458 143.15)
 		(end 130.844699 143.15)
@@
 	)
 	(segment
-		(start 121.599975 101.75)
-		(end 120.424573 102.064947)
-		(width 0.25)
-		(layer "B.Cu")
-		(net 4)
-	)
-	(segment
 		(start 127.5276 126.0905)
 		(end 128.3466 126.0905)
@@
 	)
 	(segment
-		(start 114.1873 106.8727)
-		(end 114.1873 107.4004)
-		(width 0.1016)
-		(layer "B.Cu")
-		(net 5)
-	)
-	(segment
 		(start 124.4748 113.6332)
 		(end 124.7873 113.3207)
@@
 	)
 	(segment
-		(start 113.6604 107.9273)
-		(end 112.7279 107.9273)
-		(width 0.1016)
-		(layer "B.Cu")
-		(net 5)
-	)
-	(segment
 		(start 124.3278 122.3863)
 		(end 124.6195 122.3863)
@@
 	)
 	(segment
-		(start 111.1888 109.4664)
+		(start 111.1888 109.4663)
 		(end 111.1888 116.6388)
 		(width 0.1016)
@@
 	)
 	(segment
-		(start 125.0267 112.8813)
-		(end 125.0267 112.8272)
-		(width 0.1016)
-		(layer "B.Cu")
-		(net 5)
-	)
-	(segment
 		(start 111.660562 123.249482)
 		(end 112.300562 123.889482)
@@
 	)
 	(segment
-		(start 112.7279 107.9273)
-		(end 111.1888 109.4664)
-		(width 0.1016)
-		(layer "B.Cu")
-		(net 5)
-	)
-	(segment
 		(start 123.78125 136.61875)
 		(end 123.78125 136.68125)
@@
 	)
 	(segment
-		(start 114.1873 107.4004)
-		(end 113.6604 107.9273)
-		(width 0.1016)
-		(layer "B.Cu")
-		(net 5)
-	)
-	(segment
 		(start 125.65625 133.05625)
 		(end 124.09375 133.05625)
@@
 	)
 	(segment
-		(start 102.53125 137.99375)
+		(start 102.53125 137.211515)
 		(end 102.53125 134.80625)
 		(width 0.1016)
@@
 	)
 	(segment
-		(start 135.88 124.43)
-		(end 135.88 126)
-		(width 0.15)
-		(layer "B.Cu")
-		(net 6)
-	)
-	(segment
 		(start 122.1244 111.9341)
 		(end 122.1244 112.4175)
@@
 	)
 	(segment
-		(start 116.043 135.5)
-		(end 116.043 138.4)
-		(width 0.35)
-		(layer "B.Cu")
-		(net 133)
-	)
-	(segment
 		(start 137.853 140.9082)
 		(end 136.5571 140.9082)
@@
 	)
 	(segment
+		(start 114.1873 106.8727)
+		(end 114.02 105.55)
+		(width 0.2)
+		(layer "B.Cu")
+		(net 140)
+	)
+	(segment
 		(start 113.8708 105.4008)
 		(end 111.739 105.4008)
@@
 	)
 	(zone
-		(net 4)
-		(net_name "+5V")
+		(net 3)
+		(net_name "VBAT")
 		(layer "In4.Cu")
 		(hatch edge 0.5)
-		(priority 13)
+		(priority 15)
 		(connect_pads yes
 			(clearance 0.25)
@@
 		(polygon
 			(pts
-				(xy 110 134) (xy 115 134) (xy 115 138) (xy 110 138)
+				(xy 133.5 117.5) (xy 136.5 117.5) (xy 136.5 124.5) (xy 133.5 124.5)
 			)
 		)
@@
 		(layer "In4.Cu")
 		(hatch edge 0.5)
-		(priority 15)
+		(priority 4)
 		(connect_pads yes
 			(clearance 0.25)
@@
 		(polygon
 			(pts
-				(xy 133.5 117.5) (xy 136.5 117.5) (xy 136.5 124.5) (xy 133.5 124.5)
+				(xy 115.5 105) (xy 120.6 105) (xy 120.6 116) (xy 115.5 116)
 			)
 		)
 	)
 	(zone
-		(net 3)
-		(net_name "VBAT")
+		(net 6)
+		(net_name "+3V3A")
 		(layer "In4.Cu")
 		(hatch edge 0.5)
-		(priority 4)
+		(priority 3)
 		(connect_pads yes
 			(clearance 0.25)
@@
 		(polygon
 			(pts
-				(xy 115.5 105) (xy 120.6 105) (xy 120.6 116) (xy 115.5 116)
+				(xy 101 135.5) (xy 108.2 135.5) (xy 108.2 145) (xy 101 145)
 			)
 		)
 	)
 	(zone
-		(net 6)
-		(net_name "+3V3A")
+		(net 3)
+		(net_name "VBAT")
 		(layer "In4.Cu")
 		(hatch edge 0.5)
-		(priority 3)
+		(priority 1)
 		(connect_pads yes
 			(clearance 0.25)
@@
 		(polygon
 			(pts
-				(xy 101 135.5) (xy 108.2 135.5) (xy 108.2 145) (xy 101 145)
+				(xy 101 104) (xy 106.5 104) (xy 106.5 119) (xy 101 119)
 			)
 		)
 	)
 	(zone
-		(net 3)
-		(net_name "VBAT")
+		(net 6)
+		(net_name "+3V3A")
 		(layer "In4.Cu")
 		(hatch edge 0.5)
-		(priority 1)
+		(priority 9)
 		(connect_pads yes
 			(clearance 0.25)
@@
 		(polygon
 			(pts
-				(xy 101 104) (xy 106.5 104) (xy 106.5 119) (xy 101 119)
+				(xy 107.5 143.4) (xy 118 143.4) (xy 118 144.6) (xy 107.5 144.6)
 			)
 		)
@@
 		(polygon
 			(pts
-				(xy 115.5 109) (xy 118 109) (xy 118 126) (xy 115.5 126)
+				(xy 115.5 109) (xy 118 109) (xy 118 113.4) (xy 115.5 113.4)
 			)
 		)
@@
 	)
 	(zone
+		(net 6)
+		(net_name "+3V3A")
+		(layer "In4.Cu")
+		(hatch edge 0.5)
+		(priority 13)
+		(connect_pads yes
+			(clearance 0.25)
+		)
+		(min_thickness 0.2)
+		(filled_areas_thickness no)
+		(fill yes
+			(thermal_gap 0.5)
+			(thermal_bridge_width 0.5)
+		)
+		(polygon
+			(pts
+				(xy 103.9 111.8) (xy 106.5 111.8) (xy 106.5 113.4) (xy 105.6 113.4) (xy 105.6 126.5) (xy 103.9 126.5)
+			)
+		)
+	)
+	(zone
 		(net 4)
 		(net_name "+5V")
@@
 		(polygon
 			(pts
-				(xy 112 120) (xy 116.5 120) (xy 116.5 135.5) (xy 112 135.5)
+				(xy 112 120) (xy 116.3 120) (xy 116.3 120.3) (xy 127 120.3) (xy 127 119.95) (xy 128.3 119.95) (xy 128.3 121.9)
+				(xy 119.4 121.9) (xy 119.4 122.75) (xy 118.3 122.75) (xy 118.3 121.9) (xy 116.5 121.9) (xy 116.5 135)
+				(xy 117 135) (xy 117 141.3) (xy 110.2 141.3) (xy 110.2 136.3) (xy 107.8 136.3) (xy 107.8 135) (xy 112 135)
 			)
 		)
@@
 	)
 	(zone
-		(net 4)
-		(net_name "+5V")
+		(net 3)
+		(net_name "VBAT")
 		(layer "In4.Cu")
 		(hatch edge 0.5)
-		(priority 20)
+		(priority 3)
 		(connect_pads yes
 			(clearance 0.25)
@@
 		(polygon
 			(pts
-				(xy 126 135.5) (xy 141 135.5) (xy 141 142) (xy 126 142)
+				(xy 116 113.4) (xy 131.3 113.4) (xy 131.3 117.8) (xy 116 117.8)
 			)
 		)
@@
 		(layer "In4.Cu")
 		(hatch edge 0.5)
-		(priority 12)
+		(priority 20)
 		(connect_pads yes
 			(clearance 0.25)
@@
 		(polygon
 			(pts
-				(xy 106.5 132.5) (xy 112 132.5) (xy 112 135.4) (xy 106.5 135.4)
+				(xy 126 135.5) (xy 141 135.5) (xy 141 142) (xy 126 142)
 			)
 		)
@@
 		(polygon
 			(pts
-				(xy 115.23 109.25) (xy 126.15 109.25) (xy 126.15 115.66) (xy 115.23 115.66)
+				(xy 115.2 109.2) (xy 126.2 109.2) (xy 126.2 113.4) (xy 115.2 113.4)
 			)
 		)

Commit message: fit 47 nF on the MAX2112 offset caps, as the datasheet asks
Parts:
- C61, C63: value 100n -> 47n
Changed lines of the file:
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@@
 			)
 		)
-		(property "Value" "100n"
+		(property "Value" "47n"
 			(at 0 -1.16 180)
 			(layer "B.Fab")
@@
 			)
 		)
-		(property "Value" "100n"
+		(property "Value" "47n"
 			(at 0 -1.16 180)
 			(layer "B.Fab")
