File: NAVCORE-SoOP.kicad_pcb (KiCad board)
At the start: 6 copper layers, 45 x 47.2 mm, 195 parts, among them J1 USB-C, J11 SERIAL2 4P, J12 U.FL ANT, J14 FLOW 6P, J15 LED 3P, J16 BUZZ 2P, J17 SERVO 6P, J18 PYRO 2P, J19 SWD 4P, J2 ESC 8P, J20 TOUCH 2P, J3 GPS+I2C, J5 RC IN, J6 CAN 4P, J8 microSD, J9 I2C 4P, P41 TEL_5V, P44 TEL_PPS, P46 TEL_GND, P71 RF_5V, P72 RF_TX, P73 RF_RX, P74 RF_GND, Q1 AO3400A, Q3 AO3400A, Q4 WST4041, Q5 AO3400A, SW1 BOOT, SW2 RESET, U1 STM32H743VIT6, U10 TLV75533, U11 SN65HVD230, U12 USBLC6-2SC6, U13 MAX2112, U14 OPA2374, U17 74LVC1G17, U19 TMP119, U2 ICM-42688-P, U20 LMR33630A, U21 XC6206P332MR, U3 ICM-42605, U4 MS5611, U5 W25Q128JVSIQ, U8 LMR33630A, U9 AP2112K-3.3, Y1 8MHz, Y2 25MHz TCXO

Commit message: widen C29 to 2u2 and sync the LCSC properties
Parts:
- C29: value 1u -> 2u2
Changed lines of the file:
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@@
 			)
 		)
-		(property "Value" "1u"
+		(property "Value" "2u2"
 			(at 0 1.16 0)
 			(layer "F.Fab")
@@
 			)
 		)
-		(property "LCSC" "C52923"
+		(property "LCSC" "C12530"
 			(at 0 0 0)
 			(layer "F.SilkS")

Commit message: hold the pyro gate down with 10 nF, load-test the bucks on the bench
Parts:
- added C87: 10n, Capacitor_SMD:C_0402_1005Metric, F.Cu at (105.5, 134.9)
Routing:
- net PYRO_GATE: track 2.74 -> 5.54 mm, vias 0 -> 2
Changed lines of the file:
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@@
 		)
 	)
+	(footprint "Capacitor_SMD:C_0402_1005Metric"
+		(layer "F.Cu")
+		(at 105.5 134.9)
+		(descr "Capacitor SMD 0402 (1005 Metric), square (rectangular) end terminal, IPC-7351 nominal, (Body size source: IPC-SM-782 page 76, https://www.pcb-3d.com/wordpress/wp-content/uploads/ipc-sm-782a_amendment_1_and_2.pdf), generated with kicad-footprint-generator")
+		(tags "capacitor")
+		(property "Reference" "C87"
+			(at 0 -1.16 0)
+			(layer "F.Fab")
+			(effects
+				(font
+					(size 1 1)
+					(thickness 0.15)
+				)
+			)
+		)
+		(property "Value" "10n"
+			(at 0 1.16 0)
+			(layer "F.Fab")
+			(effects
+				(font
+					(size 1 1)
+					(thickness 0.15)
+				)
+			)
+		)
+		(property "Datasheet" ""
+			(at 0 0 0)
+			(layer "F.Fab")
+			(hide yes)
+			(effects
+				(font
+					(size 1.27 1.27)
+					(thickness 0.15)
+				)
+			)
+		)
+		(property "Description" ""
+			(at 0 0 0)
+			(layer "F.Fab")
+			(hide yes)
+			(effects
+				(font
+					(size 1.27 1.27)
+					(thickness 0.15)
+				)
+			)
+		)
+		(attr smd)
+		(fp_line
+			(start -0.107836 -0.36)
+			(end 0.107836 -0.36)
+			(stroke
+				(width 0.12)
+				(type solid)
+			)
+			(layer "F.SilkS")
+		)
+		(fp_line
+			(start -0.107836 0.36)
+			(end 0.107836 0.36)
+			(stroke
+				(width 0.12)
+				(type solid)
+			)
+			(layer "F.SilkS")
+		)
+		(fp_rect
+			(start -0.91 -0.46)
+			(end 0.91 0.46)
+			(stroke
+				(width 0.05)
+				(type solid)
+			)
+			(fill no)
+			(layer "F.CrtYd")
+		)
+		(fp_rect
+			(start -0.5 -0.25)
+			(end 0.5 0.25)
+			(stroke
+				(width 0.1)
+				(type solid)
+			)
+			(fill no)
+			(layer "F.Fab")
+		)
+		(fp_text user "${REFERENCE}"
+			(at 0 0 0)
+			(layer "F.Fab")
+			(effects
+				(font
+					(size 0.25 0.25)
+					(thickness 0.04)
+				)
+			)
+		)
+		(pad "1" smd roundrect
+			(at -0.48 0)
+			(size 0.56 0.62)
+			(layers "F.Cu" "F.Mask" "F.Paste")
+			(roundrect_rratio 0.25)
+			(net 144 "PYRO_GATE")
+		)
+		(pad "2" smd roundrect
+			(at 0.48 0)
+			(size 0.56 0.62)
+			(layers "F.Cu" "F.Mask" "F.Paste")
+			(roundrect_rratio 0.25)
+			(net 1 "GND")
+		)
+		(embedded_fonts no)
+		(model "${JLC_LIB}/packages3d/C_0402_1005Metric.step"
+			(offset
+				(xyz -0.55 -0.3 0)
+			)
+			(scale
+				(xyz 1 1 1)
+			)
+			(rotate
+				(xyz 0 0 0)
+			)
+		)
+	)
 	(footprint "jlc:SOIC-8_L5.3-W5.3-P1.27-LS8.0-BL"
 		(layer "F.Cu")
@@
 	)
 	(segment
+		(start 105.02 134.9)
+		(end 104.9 135)
+		(width 0.1016)
+		(layer "F.Cu")
+		(net 144)
+	)
+	(segment
 		(start 102.01 138.5)
 		(end 102.99 138.5)
@@
 	)
 	(segment
+		(start 104.9 135)
+		(end 104.9 135.2)
+		(width 0.1016)
+		(layer "F.Cu")
+		(net 144)
+	)
+	(segment
 		(start 103.5 137.4291)
 		(end 103.5 136.95)
@@
 		(net 144)
 	)
+	(via
+		(at 104.9 135.2)
+		(size 0.45)
+		(drill 0.2)
+		(layers "F.Cu" "B.Cu")
+		(net 144)
+	)
+	(via
+		(at 103.5 136.95)
+		(size 0.45)
+		(drill 0.2)
+		(layers "F.Cu" "B.Cu")
+		(net 144)
+	)
+	(segment
+		(start 104.5 136.1)
+		(end 104.45 136.15)
+		(width 0.1016)
+		(layer "In2.Cu")
+		(net 144)
+	)
+	(segment
+		(start 103.7 136.95)
+		(end 103.5 136.95)
+		(width 0.1016)
+		(layer "In2.Cu")
+		(net 144)
+	)
+	(segment
+		(start 104.45 136.2)
+		(end 103.7 136.95)
+		(width 0.1016)
+		(layer "In2.Cu")
+		(net 144)
+	)
+	(segment
+		(start 104.9 135.2)
+		(end 104.5 135.6)
+		(width 0.1016)
+		(layer "In2.Cu")
+		(net 144)
+	)
+	(segment
+		(start 104.45 136.15)
+		(end 104.45 136.2)
+		(width 0.1016)
+		(layer "In2.Cu")
+		(net 144)
+	)
+	(segment
+		(start 104.5 135.6)
+		(end 104.5 136.1)
+		(width 0.1016)
+		(layer "In2.Cu")
+		(net 144)
+	)
