File: NAVCORE-SoOP.kicad_sch (KiCad schematic)
At the start: 195 parts, among them J1 USB-C, J11 SERIAL2 4P, J12 MMCX-KWE-90, J14 FLOW 6P, J17 SERVO1, J19 TC2030-NL, J2 ESC 8P, J21 COMPANION, J22 PAYLOAD 5V, J23 SERVO2, J3 GPS+I2C, J5 RC IN, J6 CAN 4P, J8 microSD, J9 I2C 4P, P151 LED_5V, P152 LED_DIN, P153 LED_GND, P161 BUZ_5V, P162 BUZ_OUT, P163 BUZ_GND, Q1 AO3400A, Q3 AO3400A, Q4 WST4041, SW1 BOOT, SW2 RESET, U1 STM32H743VIT6, U10 TLV75533, U11 SN65HVD230, U12 USBLC6-2SC6, U13 MAX2112, U14 OPA2374, U17 74LVC1G17, U19 TMP119, U2 ICM-42688-P, U20 LMR33630A, U21 XC6206P332MR, U22 SRV05-4, U23 SRV05-4, U24 AP22653, U25 INA180A2, U3 ICM-42605, U4 MS5611, U5 W25Q128JVPIQ, U8 LMR33630A, U9 TLV75733P, Y1 8MHz, Y2 25MHz TCXO

Commit message: route Rev D and build its fab outputs
Parts:
- J2: LCSC C265111 -> C42376901
Changed lines of the file:
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@@
 		(property "Value" "ESC 8P" (at 397.51 58.42 0) (effects (font (size 1.27 1.27)) (justify left)))
 		(property "Footprint" "jlc:CONN-SMD_SM08B-GHS-TB-LF-SN" (at 397.51 60.96 0) (effects (font (size 1.27 1.27)) hide))
-		(property "LCSC" "C265111" (at 397.51 60.96 0) (effects (font (size 1.27 1.27)) hide))
+		(property "LCSC" "C42376901" (at 397.51 60.96 0) (effects (font (size 1.27 1.27)) hide))
 		(pin "1")
 		(pin "2")

Commit message: respin design: clamps on every port, Remote ID and a tested MAX2112 setup
Parts:
- added D9: PESD5V0C1BSF, jlc:DSN0603-2_L0.6-W0.3-P0.40-BI, symbol Device:D_TVS
- added R70, R72, R73, R74, R75: 100R, Resistor_SMD:R_0402_1005Metric, symbol Device:R
- added R71: 2k2, Resistor_SMD:R_0402_1005Metric, symbol Device:R
- added RN1: 33R x4, Resistor_SMD:R_Array_Convex_4x0402, symbol Device:R_Pack04
- added U26, U27, U28, U29, U30: TPD4E05U06, Package_SON:USON-10_2.5x1.0mm_P0.5mm, symbol Power_Protection:TPD4E05U06DQA
Connections:
- net ESC_CUR: now also R71.2; no longer J2.7
- net ESC_TEL: now also R70.2; no longer J2.8
- net EXT_CS1: now also U1.7 (PC13); no longer U1.85 (PD4)
- net GND: now also D9.2 (A2)
- net M1: now also RN1.4 (R4.1); no longer J2.3
- net M2: now also RN1.3 (R3.1); no longer J2.4
- net M3: now also RN1.2 (R2.1); no longer J2.5
- net M4: now also RN1.1 (R1.1); no longer J2.6
- net PWM5: now also U1.96 (PB9); no longer U1.24 (PA2)
- net PWM7: now also U1.95 (PB8), R75.2; no longer J17.1, U1.59 (PD12)
- net PWM8: now also R74.2; no longer J23.1
- net USART1_RX: now also R73.2; no longer J11.3
- net USART1_TX: now also R72.2; no longer J11.2
- new net ESC_CUR_J: J2.7, R71.1
- new net ESC_TEL_J: J2.8, R70.1
- new net M1_J: J2.3, RN1.5 (R4.2)
- new net M2_J: J2.4, RN1.6 (R3.2)
- new net M3_J: J2.5, RN1.7 (R2.2)
- new net M4_J: J2.6, RN1.8 (R1.2)
- new net PWM7_J: D9.1 (A1), J17.1, R75.1
- new net PWM8_J: J23.1, R74.1
- new net USART1_RX_J: J11.3, R73.1
- new net USART1_TX_J: J11.2, R72.1
- no-connect marks 44 -> 50

Commit message: fix the schematic export
Connections:
- net ESC_CUR_J: now also U27.1 (D1+), U27.10 (NC)
- net ESC_TEL_J: now also U27.2 (D1-), U27.9 (NC)
- net EXT_CS1: now also U29.5 (D2-), U29.6 (NC)
- net GND: now also U26.3 (GND), U26.8 (GND), U27.3 (GND), U27.8 (GND), U28.3 (GND), U28.8 (GND), U29.3 (GND), U29.8 (GND), U30.3 (GND), U30.8 (GND)
- net M1_J: now also U26.1 (D1+), U26.10 (NC)
- net M2_J: now also U26.2 (D1-), U26.9 (NC)
- net M3_J: now also U26.4 (D2+), U26.7 (NC)
- net M4_J: now also U26.5 (D2-), U26.6 (NC)
- net PWM8_J: now also U30.4 (D2+), U30.7 (NC)
- net SPI3_MISO: now also U29.2 (D1-), U29.9 (NC)
- net SPI3_MOSI: now also U29.4 (D2+), U29.7 (NC)
- net SPI3_SCK: now also U29.1 (D1+), U29.10 (NC)
- net UART7_CTS: now also U28.4 (D2+), U28.7 (NC)
- net UART7_RTS: now also U28.5 (D2-), U28.6 (NC)
- net UART7_RX: now also U28.2 (D1-), U28.9 (NC)
- net UART7_TX: now also U28.1 (D1+), U28.10 (NC)
- net USART1_RX_J: now also U30.2 (D1-), U30.9 (NC)
- net USART1_TX_J: now also U30.1 (D1+), U30.10 (NC)
